Commit message: Autosave

File: description/gazebo_control.xacro (robot description, xacro)
@@ -3,11 +3,7 @@
     <gazebo>
         <plugin name="gazebo_ros_ackermann_drive" filename="libgazebo_ros_ackermann_drive.so">
-<!--
             <ros>
-              <namespace>demo</namespace>
-              <remapping>cmd_vel:=cmd_demo</remapping>
-              <remapping>odom:=odom_demo</remapping>
-              <remapping>distance:=distance_demo</remapping>
-            </ros> -->
+              <namespace>turjabot</namespace>
+            </ros>
             <update_rate>100.0</update_rate>
             <!-- wheels -->
@@ -27,5 +23,5 @@
             <max_speed>20</max_speed>
             <!-- PID tuning -->
-            <!-- <left_steering_pid_gain>1500 0 1</left_steering_pid_gain>
+            <left_steering_pid_gain>1500 0 1</left_steering_pid_gain>
             <left_steering_i_range>0 0</left_steering_i_range>
             <right_steering_pid_gain>1500 0 1</right_steering_pid_gain>
@@ -33,5 +29,4 @@
             <linear_velocity_pid_gain>1000 0 1</linear_velocity_pid_gain>
             <linear_velocity_i_range>0 0</linear_velocity_i_range>
-            -->
             <!-- output -->
             <publish_odom>true</publish_odom>

File: description/robot.urdf.xacro (robot description, xacro)
@@ -4,5 +4,6 @@
     <xacro:include filename="colors.xacro" />
     <xacro:include filename="robot_core.xacro" />
-    <!-- <xacro:include filename="gazebo_control.xacro" /> -->
-    <xacro:include filename="ros2_control.xacro" />
+    <xacro:include filename="gazebo_sensors.xacro" />
+    <xacro:include filename="gazebo_control.xacro" />
+    <!-- <xacro:include filename="ros2_control.xacro" /> -->
 </robot>

File: description/robot_core.xacro (robot description, xacro)
@@ -162,29 +162,4 @@
         <material>Gazebo/Black</material>
     </gazebo>
-    <joint name="traction_wheel_joint" type="continuous">
-        <parent link="chassis_back" />
-        <child link="traction_wheel" />
-        <origin xyz="${drive_wheel_offset_x} -${drive_wheel_offset_y} ${drive_wheel_offset_z}" rpy="${pi/2} 0 0" />
-        <axis xyz="0 0 -1" />
-    </joint>
-    <link name="traction_wheel">
-        <visual>
-            <geometry>
-                <cylinder length="0.01" radius="0.01" />
-            </geometry>
-            <material name="black" />
-        </visual>
-        <collision>
-            <geometry>
-                <sphere radius="0.01" />
-            </geometry>
-        </collision>
-        <xacro:inertial_cylinder mass="0.001" length="0.01" radius="0.01">
-            <origin xyz="0 0 0" rpy="0 0 0"/>
-        </xacro:inertial_cylinder>
-    </link>
-    <gazebo reference="right_drive_wheel">
-        <material>Gazebo/Black</material>
-    </gazebo>
     <!-- Chassis steer left -->
     <joint name="left_chassis_steer_joint" type="revolute">
@@ -245,30 +220,4 @@
     <gazebo reference="right_chassis_steer">
         <material>Gazebo/White</material>
-    </gazebo>
-    <joint name="steering_joint" type="revolute">
-        <parent link="chassis_front" />
-        <child link="steering_link" />
-        <origin xyz="${drive_wheel_offset_x} -${drive_wheel_offset_y} ${drive_wheel_offset_z}" rpy="${pi/2} 0 0" />
-        <axis xyz="0 0 1" />
-        <limit lower="-${steer_turnlimit}" upper="${steer_turnlimit}" velocity="100" effort="10000" />
-    </joint>
-    <link name="steering_link">
-        <visual>
-            <geometry>
-                <cylinder length="0.01" radius="0.01" />
-            </geometry>
-            <material name="black" />
-        </visual>
-        <collision>
-            <geometry>
-                <sphere radius="0.01" />
-            </geometry>
-        </collision>
-        <xacro:inertial_cylinder mass="0.001" length="0.01" radius="0.01">
-            <origin xyz="0 0 0" rpy="0 0 0"/>
-        </xacro:inertial_cylinder>
-    </link>
-    <gazebo reference="right_drive_wheel">
-        <material>Gazebo/Black</material>
     </gazebo>
     <!-- Steer wheel left -->

File: description/ros2_control.xacro (robot description, xacro)
@@ -25,14 +25,4 @@
             </state_interface>
         </joint>
-        <joint name="traction_wheel_joint">
-            <command_interface name="velocity">
-                <param name="min">-10</param>
-                <param name="max">10</param>
-            </command_interface>
-            <state_interface name="velocity" />
-            <state_interface name="position">
-                <param name="initial_value">0.0</param>
-            </state_interface>
-        </joint>
         <joint name="left_chassis_steer_joint">
             <command_interface name="position">
@@ -47,15 +37,4 @@
         </joint>
         <joint name="right_chassis_steer_joint">
-            <command_interface name="position">
-                <param name="min">-${pi/6}</param>
-                <param name="max">${pi/6}</param>
-            </command_interface>
-            <state_interface name="position">
-                <param name="initial_value">0.5</param>
-            </state_interface>
-            <state_interface name="velocity"/>
-            <state_interface name="effort"/>
-        </joint>
-        <joint name="steering_joint">
             <command_interface name="position">
                 <param name="min">-${pi/6}</param>
