Commit message: Autosave

File: description/robot.urdf.xacro (robot description, xacro)
@@ -3,4 +3,5 @@
     <!-- Example link -->
     <!-- <link name="base_link"></link> -->
+    <xacro:include filename="inertial_macros.xacro" />
     <xacro:include filename="colors.xacro" />
     <xacro:include filename="robot_core.xacro" />

File: description/robot_core.xacro (robot description, xacro)
@@ -6,9 +6,9 @@
     <xacro:property name="chassis_back_width" value="0.082"/>
     <xacro:property name="chassis_back_height" value="0.12"/>
-    <xacro:property name="chassis_back_mass" value="1.0"/>
+    <xacro:property name="chassis_back_mass" value="0.2"/>
     <xacro:property name="chassis_front_length" value="0.095"/>
     <xacro:property name="chassis_front_width" value="0.055"/>
     <xacro:property name="chassis_front_height" value="0.03"/>
-    <xacro:property name="chassis_front_mass" value="1.0"/>
+    <xacro:property name="chassis_front_mass" value="0.1"/>
     <!-- Chassis steering parts -->
     <xacro:property name="chassis_steer_length" value="0.025"/>
@@ -23,5 +23,5 @@
     <xacro:property name="wheel_radius" value="0.0325"/>
     <xacro:property name="wheel_thickness" value="0.025"/>
-    <xacro:property name="wheel_mass" value="0.05"/>
+    <xacro:property name="wheel_mass" value="0.02"/>
     <xacro:property name="drive_wheel_offset_x" value="0.06"/>
     <xacro:property name="drive_wheel_offset_y" value="${chassis_back_width/2 + wheel_thickness/2 + 0.003}"/>
@@ -34,5 +34,5 @@
     <xacro:property name="camera_pan_width" value="0.019"/>
     <xacro:property name="camera_pan_height" value="0.039"/>
-    <xacro:property name="camera_pan_mass" value="0.02"/>
+    <xacro:property name="camera_pan_mass" value="0.05"/>
     <xacro:property name="camera_pan_offset_x" value="${chassis_front_length - 0.005}"/>
     <xacro:property name="camera_pan_offset_y" value="0"/>
@@ -41,5 +41,5 @@
     <xacro:property name="camera_tilt_width" value="0.039"/>
     <xacro:property name="camera_tilt_height" value="0.047"/>
-    <xacro:property name="camera_tilt_mass" value="0.02"/>
+    <xacro:property name="camera_tilt_mass" value="0.05"/>
     <xacro:property name="camera_tilt_offset_x" value="0"/>
     <xacro:property name="camera_tilt_offset_y" value="0"/>
@@ -50,5 +50,5 @@
     <xacro:property name="grayscale_block_width" value="0.054"/>
     <xacro:property name="grayscale_block_height" value="0.007"/>
-    <xacro:property name="grayscale_block_mass" value="0.01"/>
+    <xacro:property name="grayscale_block_mass" value="0.02"/>
     <xacro:property name="grayscale_block_offset_x" value="${chassis_front_length + grayscale_block_length/2}"/>
     <xacro:property name="grayscale_block_offset_y" value="0"/>
@@ -75,4 +75,7 @@
             </geometry>
         </collision>
+        <xacro:inertial_box mass="${chassis_back_mass}" x="${chassis_back_length}" y="${chassis_back_width}" z="${chassis_back_height}">
+            <origin xyz="${chassis_back_length / 2} 0 ${chassis_back_height/2}" rpy="0 0 0" />
+        </xacro:inertial_box>
     </link>
     <!-- Chassis front -->
@@ -96,4 +99,7 @@
             </geometry>
         </collision>
+        <xacro:inertial_box mass="${chassis_front_mass}" x="${chassis_front_length}" y="${chassis_front_width}" z="${chassis_front_height}">
+            <origin xyz="${chassis_front_length / 2} 0 ${chassis_front_height/2}" rpy="0 0 0" />
+        </xacro:inertial_box>
     </link>
     <!-- Drive wheel left -->
@@ -116,4 +122,7 @@
             </geometry>
         </collision>
+        <xacro:inertial_cylinder mass="${wheel_mass}" length="${wheel_thickness}" radius="${wheel_radius}">
+            <origin xyz="0 0 0" rpy="0 0 0"/>
+        </xacro:inertial_cylinder>
     </link>
     <!-- Drive wheel right -->
@@ -136,4 +145,7 @@
             </geometry>
         </collision>
+        <xacro:inertial_cylinder mass="${wheel_mass}" length="${wheel_thickness}" radius="${wheel_radius}">
+            <origin xyz="0 0 0" rpy="0 0 0"/>
+        </xacro:inertial_cylinder>
     </link>
     <!-- Chassis steer left -->
@@ -159,4 +171,7 @@
             </geometry>
         </collision>
+        <xacro:inertial_box mass="${chassis_steer_mass}" x="${chassis_steer_length}" y="${chassis_steer_width}" z="${chassis_steer_height}">
+            <origin xyz="${steer_wheel_offset_x} 0 0" rpy="0 0 0" />
+        </xacro:inertial_box>
     </link>
     <!-- Chassis steer right -->
@@ -182,4 +197,7 @@
             </geometry>
         </collision>
+        <xacro:inertial_box mass="${chassis_steer_mass}" x="${chassis_steer_length}" y="${chassis_steer_width}" z="${chassis_steer_height}">
+            <origin xyz="${steer_wheel_offset_x} 0 0" rpy="0 0 0" />
+        </xacro:inertial_box>
     </link>
     <!-- Steer wheel left -->
@@ -202,4 +220,7 @@
             </geometry>
         </collision>
+        <xacro:inertial_cylinder mass="${wheel_mass}" length="${wheel_thickness}" radius="${wheel_radius}">
+            <origin xyz="0 0 0" rpy="0 0 0"/>
+        </xacro:inertial_cylinder>
     </link>
     <!-- Steer wheel right -->
@@ -222,4 +243,7 @@
             </geometry>
         </collision>
+        <xacro:inertial_cylinder mass="${wheel_mass}" length="${wheel_thickness}" radius="${wheel_radius}">
+            <origin xyz="0 0 0" rpy="0 0 0"/>
+        </xacro:inertial_cylinder>
     </link>
     <!-- Camera tower pan -->
@@ -245,4 +269,7 @@
             </geometry>
         </collision>
+        <xacro:inertial_box mass="${camera_pan_mass}" x="${camera_pan_length}" y="${camera_pan_width}" z="${camera_pan_height}">
+            <origin xyz="${-0.022 + camera_pan_length/2} 0 ${camera_pan_height/2}" />
+        </xacro:inertial_box>
     </link>
     <!-- Camera tower tilt -->
@@ -268,4 +295,7 @@
             </geometry>
         </collision>
+        <xacro:inertial_box mass="${camera_tilt_mass}" x="${camera_tilt_length}" y="${camera_tilt_width}" z="${camera_tilt_height}">
+            <origin xyz="${-0.014 + camera_tilt_length/2} 0 ${-0.017 + camera_tilt_height/2}" />
+        </xacro:inertial_box>
     </link>
     <!-- Grayscale sensor block -->
@@ -287,4 +317,7 @@
             </geometry>
         </collision>
+        <xacro:inertial_box mass="${grayscale_block_mass}" x="${grayscale_block_length}" y="${grayscale_block_width}" z="${grayscale_block_height}">
+            <origin xyz="0 0 0" />
+        </xacro:inertial_box>
     </link>
 </robot>

Commit message: Autosave

File: description/robot.urdf.xacro (robot description, xacro)
@@ -6,3 +6,4 @@
     <xacro:include filename="colors.xacro" />
     <xacro:include filename="robot_core.xacro" />
+    <xacro:include filename="gazebo_control.xacro" />
 </robot>

File: description/robot_core.xacro (robot description, xacro)
@@ -79,4 +79,7 @@
         </xacro:inertial_box>
     </link>
+    <gazebo reference="chassis_back">
+        <material>Gazebo/White</material>
+    </gazebo>
     <!-- Chassis front -->
     <joint name="chassis_front_joint" type="fixed">
@@ -103,4 +106,7 @@
         </xacro:inertial_box>
     </link>
+    <gazebo reference="chassis_front">
+        <material>Gazebo/White</material>
+    </gazebo>
     <!-- Drive wheel left -->
     <joint name="left_drive_wheel_joint" type="continuous">
@@ -126,4 +132,7 @@
         </xacro:inertial_cylinder>
     </link>
+    <gazebo reference="left_drive_wheel">
+        <material>Gazebo/Black</material>
+    </gazebo>
     <!-- Drive wheel right -->
     <joint name="right_drive_wheel_joint" type="continuous">
@@ -149,4 +158,7 @@
         </xacro:inertial_cylinder>
     </link>
+    <gazebo reference="right_drive_wheel">
+        <material>Gazebo/Black</material>
+    </gazebo>
     <!-- Chassis steer left -->
     <joint name="left_chassis_steer_joint" type="revolute">
@@ -175,4 +187,7 @@
         </xacro:inertial_box>
     </link>
+    <gazebo reference="left_chassis_steer">
+        <material>Gazebo/White</material>
+    </gazebo>
     <!-- Chassis steer right -->
     <joint name="right_chassis_steer_joint" type="revolute">
@@ -201,4 +216,7 @@
         </xacro:inertial_box>
     </link>
+    <gazebo reference="right_chassis_steer">
+        <material>Gazebo/White</material>
+    </gazebo>
     <!-- Steer wheel left -->
     <joint name="left_steer_wheel_joint" type="continuous">
@@ -224,4 +242,7 @@
         </xacro:inertial_cylinder>
     </link>
+    <gazebo reference="left_steer_wheel">
+        <material>Gazebo/Black</material>
+    </gazebo>
     <!-- Steer wheel right -->
     <joint name="right_steer_wheel_joint" type="continuous">
@@ -247,4 +268,7 @@
         </xacro:inertial_cylinder>
     </link>
+    <gazebo reference="right_steer_wheel">
+        <material>Gazebo/Black</material>
+    </gazebo>
     <!-- Camera tower pan -->
     <joint name="camera_pan_joint" type="revolute">
@@ -273,4 +297,7 @@
         </xacro:inertial_box>
     </link>
+    <gazebo reference="camera_pan">
+        <material>Gazebo/White</material>
+    </gazebo>
     <!-- Camera tower tilt -->
     <joint name="camera_tilt_joint" type="revolute">
@@ -299,4 +326,7 @@
         </xacro:inertial_box>
     </link>
+    <gazebo reference="camera_tilt">
+        <material>Gazebo/White</material>
+    </gazebo>
     <!-- Grayscale sensor block -->
     <joint name="grayscale_block_joint" type="fixed">
@@ -321,3 +351,6 @@
         </xacro:inertial_box>
     </link>
+    <gazebo reference="grayscale_block">
+        <material>Gazebo/White</material>
+    </gazebo>
 </robot>

Commit message: Autosave

File: description/robot.urdf.xacro (robot description, xacro)
@@ -6,4 +6,5 @@
     <xacro:include filename="colors.xacro" />
     <xacro:include filename="robot_core.xacro" />
-    <xacro:include filename="gazebo_control.xacro" />
+    <!-- <xacro:include filename="gazebo_control.xacro" /> -->
+    <xacro:include filename="ros2_control.xacro" />
 </robot>

File: description/robot_core.xacro (robot description, xacro)
@@ -137,4 +137,5 @@
     <!-- Drive wheel right -->
     <joint name="right_drive_wheel_joint" type="continuous">
+        <mimic joint="left_drive_wheel_joint"/>
         <parent link="chassis_back" />
         <child link="right_drive_wheel" />
@@ -192,4 +193,5 @@
     <!-- Chassis steer right -->
     <joint name="right_chassis_steer_joint" type="revolute">
+        <mimic joint="left_chassis_steer_joint"/>
         <parent link="chassis_front" />
         <child link="right_chassis_steer" />

Commit message: Autosave

File: description/robot.urdf.xacro (robot description, xacro)
@@ -1,6 +1,4 @@
 <?xml version="1.0"?>
 <robot xmlns:xacro="http://www.ros.org/wiki/xacro"  name="robot">
-    <!-- Example link -->
-    <!-- <link name="base_link"></link> -->
     <xacro:include filename="inertial_macros.xacro" />
     <xacro:include filename="colors.xacro" />

File: description/robot_core.xacro (robot description, xacro)
@@ -125,5 +125,5 @@
         <collision>
             <geometry>
-                <cylinder length="${wheel_thickness}" radius="${wheel_radius}" />
+                <sphere radius="${wheel_radius}" />
             </geometry>
         </collision>
@@ -152,8 +152,33 @@
         <collision>
             <geometry>
-                <cylinder length="${wheel_thickness}" radius="${wheel_radius}" />
+                <sphere radius="${wheel_radius}" />
             </geometry>
         </collision>
         <xacro:inertial_cylinder mass="${wheel_mass}" length="${wheel_thickness}" radius="${wheel_radius}">
+            <origin xyz="0 0 0" rpy="0 0 0"/>
+        </xacro:inertial_cylinder>
+    </link>
+    <gazebo reference="right_drive_wheel">
+        <material>Gazebo/Black</material>
+    </gazebo>
+    <joint name="traction_wheel_joint" type="continuous">
+        <parent link="chassis_back" />
+        <child link="traction_wheel" />
+        <origin xyz="${drive_wheel_offset_x} -${drive_wheel_offset_y} ${drive_wheel_offset_z}" rpy="${pi/2} 0 0" />
+        <axis xyz="0 0 -1" />
+    </joint>
+    <link name="traction_wheel">
+        <visual>
+            <geometry>
+                <cylinder length="0.01" radius="0.01" />
+            </geometry>
+            <material name="black" />
+        </visual>
+        <collision>
+            <geometry>
+                <sphere radius="0.01" />
+            </geometry>
+        </collision>
+        <xacro:inertial_cylinder mass="0.001" length="0.01" radius="0.01">
             <origin xyz="0 0 0" rpy="0 0 0"/>
         </xacro:inertial_cylinder>
@@ -168,5 +193,5 @@
         <origin xyz="${chassis_steer_offset_x} ${chassis_steer_offset_y} ${chassis_steer_offset_z}" />
         <axis xyz="0 0 1" />
-        <limit lower="-${steer_turnlimit}" upper="${steer_turnlimit}" velocity="100" effort="100" />
+        <limit lower="-${steer_turnlimit}" upper="${steer_turnlimit}" velocity="100" effort="10000" />
     </joint>
     <link name="left_chassis_steer">
@@ -198,5 +223,5 @@
         <origin xyz="${chassis_steer_offset_x} -${chassis_steer_offset_y} ${chassis_steer_offset_z}" />
         <axis xyz="0 0 1" />
-        <limit lower="-${steer_turnlimit}" upper="${steer_turnlimit}" velocity="100" effort="100" />
+        <limit lower="-${steer_turnlimit}" upper="${steer_turnlimit}" velocity="100" effort="10000" />
     </joint>
     <link name="right_chassis_steer">
@@ -220,4 +245,30 @@
     <gazebo reference="right_chassis_steer">
         <material>Gazebo/White</material>
+    </gazebo>
+    <joint name="steering_joint" type="revolute">
+        <parent link="chassis_front" />
+        <child link="steering_link" />
+        <origin xyz="${drive_wheel_offset_x} -${drive_wheel_offset_y} ${drive_wheel_offset_z}" rpy="${pi/2} 0 0" />
+        <axis xyz="0 0 1" />
+        <limit lower="-${steer_turnlimit}" upper="${steer_turnlimit}" velocity="100" effort="10000" />
+    </joint>
+    <link name="steering_link">
+        <visual>
+            <geometry>
+                <cylinder length="0.01" radius="0.01" />
+            </geometry>
+            <material name="black" />
+        </visual>
+        <collision>
+            <geometry>
+                <sphere radius="0.01" />
+            </geometry>
+        </collision>
+        <xacro:inertial_cylinder mass="0.001" length="0.01" radius="0.01">
+            <origin xyz="0 0 0" rpy="0 0 0"/>
+        </xacro:inertial_cylinder>
+    </link>
+    <gazebo reference="right_drive_wheel">
+        <material>Gazebo/Black</material>
     </gazebo>
     <!-- Steer wheel left -->
@@ -237,5 +288,5 @@
         <collision>
             <geometry>
-                <cylinder length="${wheel_thickness}" radius="${wheel_radius}" />
+                <sphere radius="${wheel_radius}" />
             </geometry>
         </collision>
@@ -263,5 +314,5 @@
         <collision>
             <geometry>
-                <cylinder length="${wheel_thickness}" radius="${wheel_radius}" />
+                <sphere radius="${wheel_radius}" />
             </geometry>
         </collision>

File: description/ros2_control.xacro (robot description, xacro)
@@ -10,5 +10,7 @@
                 <param name="max">10</param>
             </command_interface>
-            <state_interface name="position" />
+            <state_interface name="position">
+                <param name="initial_value">0.0</param>
+            </state_interface>
             <state_interface name="velocity" />
         </joint>
@@ -19,18 +21,52 @@
             </command_interface>
             <state_interface name="velocity" />
-            <state_interface name="position" />
+            <state_interface name="position">
+                <param name="initial_value">0.0</param>
+            </state_interface>
+        </joint>
+        <joint name="traction_wheel_joint">
+            <command_interface name="velocity">
+                <param name="min">-10</param>
+                <param name="max">10</param>
+            </command_interface>
+            <state_interface name="velocity" />
+            <state_interface name="position">
+                <param name="initial_value">0.0</param>
+            </state_interface>
         </joint>
         <joint name="left_chassis_steer_joint">
-            <command_interface name="position"/>
-            <state_interface name="position"/>
+            <command_interface name="position">
+                <param name="min">-${pi/6}</param>
+                <param name="max">${pi/6}</param>
+            </command_interface>
+            <state_interface name="position">
+                <param name="initial_value">0.5</param>
+            </state_interface>
             <state_interface name="velocity"/>
             <state_interface name="effort"/>
         </joint>
         <joint name="right_chassis_steer_joint">
-            <command_interface name="position"/>
-            <state_interface name="position"/>
+            <command_interface name="position">
+                <param name="min">-${pi/6}</param>
+                <param name="max">${pi/6}</param>
+            </command_interface>
+            <state_interface name="position">
+                <param name="initial_value">0.5</param>
+            </state_interface>
             <state_interface name="velocity"/>
             <state_interface name="effort"/>
         </joint>
+        <joint name="steering_joint">
+            <command_interface name="position">
+                <param name="min">-${pi/6}</param>
+                <param name="max">${pi/6}</param>
+            </command_interface>
+            <state_interface name="position">
+                <param name="initial_value">0.5</param>
+            </state_interface>
+            <state_interface name="velocity"/>
+            <state_interface name="effort"/>
+        </joint>
+<!--
         <joint name="left_steer_wheel_joint">
             <command_interface name="velocity">
@@ -48,9 +84,26 @@
             <state_interface name="velocity" />
             <state_interface name="position" />
+        </joint> -->
+<!--
+        <joint name="camera_pan_joint">
+            <command_interface name="position"/>
+            <state_interface name="position">
+                <param name="initial_value">0.0</param>
+            </state_interface>
+            <state_interface name="velocity"/>
+            <state_interface name="effort"/>
         </joint>
+        <joint name="camera_tilt_joint">
+            <command_interface name="position"/>
+            <state_interface name="position">
+                <param name="initial_value">0.0</param>
+            </state_interface>
+            <state_interface name="velocity"/>
+            <state_interface name="effort"/>
+        </joint> -->
     </ros2_control>
     <gazebo>
         <plugin name="gazebo_ros2_control" filename="libgazebo_ros2_control.so">
-            <parameters>$(find turjabot)/config/my_controllers.yaml</parameters>
+            <parameters>$(find turjabot)/config/my_controllers2.yaml</parameters>
             <!-- <parameters>$(find turjabot)/config/gaz_ros2_ctl_use_sim.yaml</parameters> -->
         </plugin>

Commit message: Autosave

File: description/robot.urdf.xacro (robot description, xacro)
@@ -4,6 +4,6 @@
     <xacro:include filename="colors.xacro" />
     <xacro:include filename="robot_core.xacro" />
-    <xacro:include filename="gazebo_sensors.xacro" />
-    <xacro:include filename="gazebo_control.xacro" />
-    <!-- <xacro:include filename="ros2_control.xacro" /> -->
+    <!-- <xacro:include filename="gazebo_sensors.xacro" />
+    <xacro:include filename="gazebo_control.xacro" /> -->
+    <xacro:include filename="ros2_control.xacro" />
 </robot>

File: description/robot_core.xacro (robot description, xacro)
@@ -302,5 +302,4 @@
         <material>Gazebo/White</material>
     </gazebo>
-    <!-- Camera tower tilt -->
     <joint name="camera_tilt_joint" type="revolute">
         <parent link="camera_pan" />

File: description/ros2_control.xacro (robot description, xacro)
@@ -10,10 +10,12 @@
                 <param name="max">10</param>
             </command_interface>
-            <state_interface name="position">
+            <!-- <state_interface name="position">
                 <param name="initial_value">0.0</param>
-            </state_interface>
+            </state_interface> -->
             <state_interface name="velocity" />
         </joint>
         <joint name="right_drive_wheel_joint">
+            <param name="mimic">left_drive_wheel_joint</param>
+            <param name="multiplier">1</param>
             <command_interface name="velocity">
                 <param name="min">-10</param>
@@ -31,10 +33,12 @@
             </command_interface>
             <state_interface name="position">
-                <param name="initial_value">0.5</param>
+                <param name="initial_value">0.0</param>
             </state_interface>
-            <state_interface name="velocity"/>
-            <state_interface name="effort"/>
+            <!-- <state_interface name="velocity"/>
+            <state_interface name="effort"/> -->
         </joint>
         <joint name="right_chassis_steer_joint">
+            <param name="mimic">left_chassis_steer_joint</param>
+            <param name="multiplier">1</param>
             <command_interface name="position">
                 <param name="min">-${pi/6}</param>
@@ -42,11 +46,10 @@
             </command_interface>
             <state_interface name="position">
-                <param name="initial_value">0.5</param>
+                <param name="initial_value">0.0</param>
             </state_interface>
             <state_interface name="velocity"/>
             <state_interface name="effort"/>
         </joint>
-<!--
-        <joint name="left_steer_wheel_joint">
+        <!--<joint name="left_steer_wheel_joint">
             <command_interface name="velocity">
                 <param name="min">-10</param>
@@ -63,6 +66,5 @@
             <state_interface name="velocity" />
             <state_interface name="position" />
-        </joint> -->
-<!--
+        </joint>-->
         <joint name="camera_pan_joint">
             <command_interface name="position"/>
@@ -70,6 +72,4 @@
                 <param name="initial_value">0.0</param>
             </state_interface>
-            <state_interface name="velocity"/>
-            <state_interface name="effort"/>
         </joint>
         <joint name="camera_tilt_joint">
@@ -78,11 +78,9 @@
                 <param name="initial_value">0.0</param>
             </state_interface>
-            <state_interface name="velocity"/>
-            <state_interface name="effort"/>
-        </joint> -->
+        </joint>
     </ros2_control>
     <gazebo>
         <plugin name="gazebo_ros2_control" filename="libgazebo_ros2_control.so">
-            <parameters>$(find turjabot)/config/my_controllers2.yaml</parameters>
+            <parameters>$(find turjabot)/config/my_controllers.yaml</parameters>
             <!-- <parameters>$(find turjabot)/config/gaz_ros2_ctl_use_sim.yaml</parameters> -->
         </plugin>
