Commit message: Autosave

File: description/ros2_control.xacro (robot description, xacro)
@@ -1,5 +1,66 @@
 <?xml version="1.0"?>
 <robot xmlns:xacro="http://www.ros.org/wiki/xacro">
-    <ros2_control name="GazeboSystem" type="system">
+<ros2_control name="Turjabot" type="system">
+        <hardware>
+            <plugin>hw_turjabot/TurjabotHardware</plugin>
+            <param name="left_drive_wheel_name">left_drive_wheel_joint</param>
+            <param name="right_drive_wheel_name">right_drive_wheel_joint</param>
+            <param name="steer_wheel_name">left_chassis_steer_joint</param>
+            <param name="camera_pan_name">camera_pan_joint</param>
+            <param name="camera_tilt_name">camera_tilt_joint</param>
+            <param name="enc_counts_per_rev">1280</param>
+        </hardware>
+        <joint name="left_drive_wheel_joint">
+            <command_interface name="velocity">
+                <param name="min">-10</param>
+                <param name="max">10</param>
+            </command_interface>
+            <state_interface name="position" />
+            <state_interface name="velocity" />
+        </joint>
+        <joint name="right_drive_wheel_joint">
+            <param name="mimic">left_drive_wheel_joint</param>
+            <param name="multiplier">1</param>
+            <command_interface name="velocity">
+                <param name="min">-10</param>
+                <param name="max">10</param>
+            </command_interface>
+            <state_interface name="position" />
+            <state_interface name="velocity" />
+        </joint>
+        <joint name="left_chassis_steer_joint">
+            <command_interface name="position">
+                <param name="min">-${pi/6}</param>
+                <param name="max">${pi/6}</param>
+            </command_interface>
+            <state_interface name="position">
+                <param name="initial_value">0.0</param>
+            </state_interface>
+        </joint>
+        <joint name="right_chassis_steer_joint">
+            <param name="mimic">left_chassis_steer_joint</param>
+            <param name="multiplier">1</param>
+            <command_interface name="position">
+                <param name="min">-${pi/6}</param>
+                <param name="max">${pi/6}</param>
+            </command_interface>
+            <state_interface name="position">
+                <param name="initial_value">0.0</param>
+            </state_interface>
+        </joint>
+        <joint name="camera_pan_joint">
+            <command_interface name="position"/>
+            <state_interface name="position">
+                <param name="initial_value">0.0</param>
+            </state_interface>
+        </joint>
+        <joint name="camera_tilt_joint">
+            <command_interface name="position"/>
+            <state_interface name="position">
+                <param name="initial_value">0.0</param>
+            </state_interface>
+        </joint>
+    </ros2_control>
+    <!-- <ros2_control name="GazeboSystem" type="system">
         <hardware>
             <plugin>gazebo_ros2_control/GazeboSystem</plugin>
@@ -10,7 +71,4 @@
                 <param name="max">10</param>
             </command_interface>
-            <!-- <state_interface name="position">
-                <param name="initial_value">0.0</param>
-            </state_interface> -->
             <state_interface name="velocity" />
         </joint>
@@ -35,6 +93,4 @@
                 <param name="initial_value">0.0</param>
             </state_interface>
-            <!-- <state_interface name="velocity"/>
-            <state_interface name="effort"/> -->
         </joint>
         <joint name="right_chassis_steer_joint">
@@ -51,20 +107,4 @@
             <state_interface name="effort"/>
         </joint>
-        <!--<joint name="left_steer_wheel_joint">
-            <command_interface name="velocity">
-                <param name="min">-10</param>
-                <param name="max">10</param>
-            </command_interface>
-            <state_interface name="position" />
-            <state_interface name="velocity" />
-        </joint>
-        <joint name="right_steer_wheel_joint">
-            <command_interface name="velocity">
-                <param name="min">-10</param>
-                <param name="max">10</param>
-            </command_interface>
-            <state_interface name="velocity" />
-            <state_interface name="position" />
-        </joint>-->
         <joint name="camera_pan_joint">
             <command_interface name="position"/>
@@ -83,6 +123,5 @@
         <plugin name="gazebo_ros2_control" filename="libgazebo_ros2_control.so">
             <parameters>$(find turjabot)/config/my_controllers.yaml</parameters>
-            <!-- <parameters>$(find turjabot)/config/gaz_ros2_ctl_use_sim.yaml</parameters> -->
         </plugin>
-    </gazebo>
+    </gazebo> -->
 </robot>
